Commit message: added joints and material

File: src/roboticarm_description/urdf/roboticArm.urdf.xacro (robot description, xacro)
@@ -10,5 +10,5 @@
   <link name="base_link">
     <visual>
-      <origin xyz="-0.035 -0.054 0" rpy="0 0 0"/>
+      <origin xyz="0 0 0" rpy="0 0 0"/>
       <geometry>
         <mesh filename="package://roboticarm_description/meshes/base_link.stl" scale="0.01 0.01 0.01"/>
@@ -24,5 +24,5 @@
   <link name="waist_link">
     <visual>
-      <origin xyz="-0.035 -0.054 0.0" rpy="0 0 0"/>
+      <origin xyz="0 0 0" rpy="0 0 0"/>
       <geometry>
         <mesh filename="package://roboticarm_description/meshes/Waist.stl" scale="0.01 0.01 0.01"/>
@@ -36,9 +36,9 @@
     <origin xyz="0 0 0" rpy="0 0 0"/>
     <axis xyz="0 0 1"/>
-    <limit lower="-3.14" upper="3.14" effort="100" velocity="1"/>
+    <limit lower="${-pi/2}" upper="${pi/2}" effort="100" velocity="1"/>
   </joint>
   <link name="arm_1_link">
     <visual>
-      <origin xyz="-0.12 0 -0.987" rpy="0 0 0"/>
+      <origin xyz="-0.14 0 -0.97" rpy="0 0 0"/>
       <geometry>
         <mesh filename="package://roboticarm_description/meshes/Arm01_1.stl" scale="0.01 0.01 0.01"/>
@@ -50,11 +50,11 @@
     <parent link="waist_link"/>
     <child link="arm_1_link"/>
-    <origin xyz="0.12 -0.08 0.987" rpy="0 0 0"/>
+    <origin xyz="0.14 0 0.97" rpy="0 0 0"/>
     <axis xyz="0 1 0"/>
-    <limit lower="-3.14" upper="3.14" effort="100" velocity="1"/>
+    <limit lower="${-pi/2}" upper="${pi/2}" effort="100" velocity="1"/>
   </joint>
   <link name="arm_2_link">
     <visual>
-      <origin xyz="0.06 -0.05 -2.08" rpy="0 0 0"/>
+      <origin xyz="-0.15 0 -2.17" rpy="0 0 0"/>
       <geometry>
         <mesh filename="package://roboticarm_description/meshes/Arm02_1.stl" scale="0.01 0.01 0.01"/>
@@ -66,11 +66,11 @@
     <parent link="arm_1_link"/>
     <child link="arm_2_link"/>
-    <origin xyz="-0.16 0.15 1.18" rpy="0 0 0"/>
+    <origin xyz="0.01 0 1.2" rpy="0 0 0"/>
     <axis xyz="0 1 0"/>
-    <limit lower="-3.14" upper="3.14" effort="100" velocity="1"/>
+    <limit lower="${-pi/2}" upper="${pi/2}" effort="100" velocity="1"/>
   </joint>
   <link name="arm_3_link">
     <visual>
-      <origin xyz="-0.82 -0.31 -2.06" rpy="0 0 0"/>
+      <origin xyz="-0.21 -0.135 -2.66" rpy="0 0 0"/>
       <geometry>
         <mesh filename="package://roboticarm_description/meshes/Arm03_1.stl" scale="0.01 0.01 0.01"/>
@@ -82,11 +82,11 @@
     <parent link="arm_2_link"/>
     <child link="arm_3_link"/>
-    <origin xyz="0.89 0.28 -0.12" rpy="0 0 0"/>
-    <axis xyz="1 0 0"/>
-    <limit lower="-3.14" upper="3.14" effort="100" velocity="1"/>
+    <origin xyz="0.05 0.11 0.5" rpy="0 0 0"/>
+    <axis xyz="0 0 1"/>
+    <limit lower="${-pi/2}" upper="${pi/2}" effort="100" velocity="1"/>
   </joint>
   <link name="gripper_base_link">
     <visual>
-      <origin xyz="-1.08 -0.32 -2.08" rpy="0 0 0"/>
+      <origin xyz="-0.15 -0.14 -3.38" rpy="0 0 0"/>
       <geometry>
         <mesh filename="package://roboticarm_description/meshes/Gripper_base.stl" scale="0.01 0.01 0.01"/>
@@ -98,13 +98,13 @@
     <parent link="arm_3_link"/>
     <child link="gripper_base_link"/>
-    <origin xyz="0.3 0 0" rpy="0 0 0"/>
+    <origin xyz="-0.05 0 0.71" rpy="0 0 0"/>
     <axis xyz="0 1 0"/>
-    <limit lower="-3.14" upper="3.14" effort="100" velocity="1"/>
+    <limit lower="${-pi/2}" upper="${pi/2}" effort="100" velocity="1"/>
   </joint>
   <link name="gear1_link">
     <visual>
-      <origin xyz="-1.5 -0.15 -2.06" rpy="0 0 0"/>
+      <origin xyz="-0.02 -0.17 -3.75" rpy="0 0 0"/>
       <geometry>
-        <mesh filename="package://roboticarm_description/meshes/gear2.stl" scale="0.01 0.01 0.01"/>
+        <mesh filename="package://roboticarm_description/meshes/gear2.002.stl" scale="0.01 0.01 0.01"/>
       </geometry>
       <material name="white"/>
@@ -114,13 +114,13 @@
     <parent link="gripper_base_link"/>
     <child link="gear1_link"/>
-    <origin xyz="0.41 -0.17 0" rpy="0 0 0"/>
-    <axis xyz="0 0 1"/>
-    <limit lower="-3.14" upper="3.14" effort="100" velocity="1"/>
+    <origin xyz="-0.14 0.03 0.37" rpy="0 0 0"/>
+    <axis xyz="1 0 0"/>
+    <limit lower="${-pi/2}" upper="${pi/2}" effort="100" velocity="1"/>
   </joint>
   <link name="gear2_link">
     <visual>
-      <origin xyz="-1.45 -0.44 -2.06" rpy="0 0 0"/>
+      <origin xyz="-0.02 0.1 -3.75" rpy="0 0 0"/>
       <geometry>
-        <mesh filename="package://roboticarm_description/meshes/gear2.001.stl" scale="0.01 0.01 0.01"/>
+        <mesh filename="package://roboticarm_description/meshes/gear2.stl" scale="0.01 0.01 0.01"/>
       </geometry>
       <material name="white"/>
@@ -130,11 +130,12 @@
     <parent link="gripper_base_link"/>
     <child link="gear2_link"/>
-    <origin xyz="0.38 0.1 0" rpy="0 0 0"/>
-    <axis xyz="0 0 1"/>
-    <limit lower="-3.14" upper="3.14" effort="100" velocity="1"/>
+    <origin xyz="-0.12 -0.245 0.366" rpy="0 0 0"/>
+    <axis xyz="1 0 0"/>
+    <mimic joint="gear1_joint" multiplier="-1.0" offset="0.0"/>
+    <limit lower="${-pi/2}" upper="${pi/2}" effort="100" velocity="1"/>
   </joint>
   <link name="finger1_link">
     <visual>
-      <origin xyz="-1.685 -0.645 -1.93" rpy="0 0 0"/>
+      <origin xyz="0.03 0.24 -4.03" rpy="0 0 0"/>
       <geometry>
         <mesh filename="package://roboticarm_description/meshes/Gripper_1.001.stl" scale="0.01 0.01 0.01"/>
@@ -143,14 +144,14 @@
     </visual>
   </link>
-  <joint name="finger1_joint" type="revolute">
-    <parent link="gripper_base_link"/>
+  <joint name="finger1_joint" type="fixed">
+    <parent link="gear2_link"/>
     <child link="finger1_link"/>
-    <origin xyz="0.62 0.295 0" rpy="0 0 0"/>
+    <origin xyz="-0.055 -0.137 0.279" rpy="0 0 0"/>
     <axis xyz="0 1 0"/>
-    <limit lower="-3.14" upper="3.14" effort="100" velocity="1"/>
+    <limit lower="${-pi/2}" upper="${pi/2}" effort="100" velocity="1"/>
   </joint>
   <link name="finger2_link">
     <visual>
-      <origin xyz="-1.77 -0.049 -1.93" rpy="0 0 0"/>
+      <origin xyz="0.03 -0.328 -4.01" rpy="0 0 0"/>
       <geometry>
         <mesh filename="package://roboticarm_description/meshes/Gripper_1.stl" scale="0.01 0.01 0.01"/>
@@ -159,10 +160,10 @@
     </visual>
   </link>
-  <joint name="finger2_joint" type="revolute">
-    <parent link="gripper_base_link"/>
+  <joint name="finger2_joint" type="fixed">
+    <parent link="gear1_link"/>
     <child link="finger2_link"/>
-    <origin xyz="0.69 -0.27 0" rpy="0 0 0"/>
+    <origin xyz="-0.055 0.162 0.26" rpy="0 0 0"/>
     <axis xyz="0 1 0"/>
-    <limit lower="-3.14" upper="3.14" effort="100" velocity="1"/>
+    <limit lower="${-pi/2}" upper="${pi/2}" effort="100" velocity="1"/>
   </joint>
 </robot>

Commit message: added launch & rviz files

File: src/roboticarm_description/urdf/roboticArm.urdf.xacro (robot description, xacro)
@@ -1,4 +1,15 @@
 <?xml version="1.0" ?>
 <robot name="Robotic" xmlns:xacro="http://www.ros.org/wiki/xacro">
+  <xacro:property name="PI" value="3.14159265359" />
+  <xacro:property name="effort" value="30" />
+  <xacro:property name="velocity" value="10" />
+  <xacro:macro name="default_inertial" params="mass">
+    <inertial>
+      <mass value="${mass}" />
+      <inertia ixx="1.0" ixy="0.0" ixz="0.0"
+                iyy="1.0" iyz="0.0"
+                izz="1.0" />
+    </inertial>
+  </xacro:macro>
   <material name="white">
     <color rgba="1.0 1.0 1.0 1.0"/>
@@ -9,4 +20,5 @@
   <link name="world"/>
   <link name="base_link">
+    <xacro:default_inertial mass="1"/>
     <visual>
       <origin xyz="0 0 0" rpy="0 0 0"/>
@@ -16,4 +28,10 @@
       <material name="white"/>
     </visual>
+    <collision>
+      <origin xyz="0 0 0" rpy="0 0 0"/>
+      <geometry>
+        <mesh filename="package://roboticarm_description/meshes/base_link.stl" scale="0.01 0.01 0.01"/>
+      </geometry>
+    </collision>
   </link>
   <joint name="base_joint" type="fixed">
@@ -23,4 +41,5 @@
   </joint>
   <link name="waist_link">
+    <xacro:default_inertial mass="0.1"/>
     <visual>
       <origin xyz="0 0 0" rpy="0 0 0"/>
@@ -30,4 +49,10 @@
       <material name="orange"/>
     </visual>
+    <collision>
+      <origin xyz="0 0 0" rpy="0 0 0"/>
+      <geometry>
+        <mesh filename="package://roboticarm_description/meshes/Waist.stl" scale="0.01 0.01 0.01"/>
+      </geometry>
+    </collision>
   </link>
   <joint name="waist_joint" type="revolute">
@@ -36,7 +61,8 @@
     <origin xyz="0 0 0" rpy="0 0 0"/>
     <axis xyz="0 0 1"/>
-    <limit lower="${-pi/2}" upper="${pi/2}" effort="100" velocity="1"/>
+    <limit lower="${-PI/2}" upper="${PI/2}" effort="${effort}" velocity="${velocity}"/>
   </joint>
   <link name="arm_1_link">
+    <xacro:default_inertial mass="0.1"/>
     <visual>
       <origin xyz="-0.14 0 -0.97" rpy="0 0 0"/>
@@ -46,4 +72,10 @@
       <material name="orange"/>
     </visual>
+    <collision>
+      <origin xyz="0 0 0" rpy="0 0 0"/>
+      <geometry>
+        <mesh filename="package://roboticarm_description/meshes/Arm01_1.stl" scale="0.01 0.01 0.01"/>
+      </geometry>
+    </collision>
   </link>
   <joint name="arm_1_joint" type="revolute">
@@ -52,7 +84,8 @@
     <origin xyz="0.14 0 0.97" rpy="0 0 0"/>
     <axis xyz="0 1 0"/>
-    <limit lower="${-pi/2}" upper="${pi/2}" effort="100" velocity="1"/>
+    <limit lower="${-PI/2}" upper="${PI/2}" effort="${effort}" velocity="${velocity}"/>
   </joint>
   <link name="arm_2_link">
+    <xacro:default_inertial mass="0.1"/>
     <visual>
       <origin xyz="-0.15 0 -2.17" rpy="0 0 0"/>
@@ -62,4 +95,10 @@
       <material name="orange"/>
     </visual>
+    <collision>
+      <origin xyz="0 0 0" rpy="0 0 0"/>
+      <geometry>
+        <mesh filename="package://roboticarm_description/meshes/Arm02_1.stl" scale="0.01 0.01 0.01"/>
+      </geometry>
+    </collision>
   </link>
   <joint name="arm_2_joint" type="revolute">
@@ -68,7 +107,8 @@
     <origin xyz="0.01 0 1.2" rpy="0 0 0"/>
     <axis xyz="0 1 0"/>
-    <limit lower="${-pi/2}" upper="${pi/2}" effort="100" velocity="1"/>
+    <limit lower="${-PI/2}" upper="${PI/2}" effort="${effort}" velocity="${velocity}"/>
   </joint>
   <link name="arm_3_link">
+    <xacro:default_inertial mass="0.1"/>
     <visual>
       <origin xyz="-0.21 -0.135 -2.66" rpy="0 0 0"/>
@@ -78,4 +118,10 @@
       <material name="orange"/>
     </visual>
+    <collision>
+      <origin xyz="0 0 0" rpy="0 0 0"/>
+      <geometry>
+        <mesh filename="package://roboticarm_description/meshes/Arm03_1.stl" scale="0.01 0.01 0.01"/>
+      </geometry>
+    </collision>
   </link>
   <joint name="arm_3_joint" type="revolute">
@@ -84,7 +130,8 @@
     <origin xyz="0.05 0.11 0.5" rpy="0 0 0"/>
     <axis xyz="0 0 1"/>
-    <limit lower="${-pi/2}" upper="${pi/2}" effort="100" velocity="1"/>
+    <limit lower="${-PI/2}" upper="${PI/2}" effort="${effort}" velocity="${velocity}"/>
   </joint>
   <link name="gripper_base_link">
+    <xacro:default_inertial mass="0.05"/>
     <visual>
       <origin xyz="-0.15 -0.14 -3.38" rpy="0 0 0"/>
@@ -94,4 +141,10 @@
       <material name="white"/>
     </visual>
+    <collision>
+      <origin xyz="0 0 0" rpy="0 0 0"/>
+      <geometry>
+        <mesh filename="package://roboticarm_description/meshes/Gripper_base.stl" scale="0.01 0.01 0.01"/>
+      </geometry>
+    </collision>
   </link>
   <joint name="gripper_base_joint" type="revolute">
@@ -100,7 +153,8 @@
     <origin xyz="-0.05 0 0.71" rpy="0 0 0"/>
     <axis xyz="0 1 0"/>
-    <limit lower="${-pi/2}" upper="${pi/2}" effort="100" velocity="1"/>
+    <limit lower="${-PI/2}" upper="${PI/2}" effort="${effort}" velocity="${velocity}"/>
   </joint>
   <link name="gear1_link">
+    <xacro:default_inertial mass="0.03"/>
     <visual>
       <origin xyz="-0.02 -0.17 -3.75" rpy="0 0 0"/>
@@ -110,4 +164,10 @@
       <material name="white"/>
     </visual>
+    <collision>
+      <origin xyz="0 0 0" rpy="0 0 0"/>
+      <geometry>
+        <mesh filename="package://roboticarm_description/meshes/gear2.002.stl" scale="0.01 0.01 0.01"/>
+      </geometry>
+    </collision>
   </link>
   <joint name="gear1_joint" type="revolute">
@@ -116,7 +176,8 @@
     <origin xyz="-0.14 0.03 0.37" rpy="0 0 0"/>
     <axis xyz="1 0 0"/>
-    <limit lower="${-pi/2}" upper="${pi/2}" effort="100" velocity="1"/>
+    <limit lower="${-PI/2}" upper="${PI/2}" effort="${effort}" velocity="${velocity}"/>
   </joint>
   <link name="gear2_link">
+    <xacro:default_inertial mass="0.03"/>
     <visual>
       <origin xyz="-0.02 0.1 -3.75" rpy="0 0 0"/>
@@ -126,4 +187,10 @@
       <material name="white"/>
     </visual>
+    <collision>
+      <origin xyz="0 0 0" rpy="0 0 0"/>
+      <geometry>
+        <mesh filename="package://roboticarm_description/meshes/gear2.stl" scale="0.01 0.01 0.01"/>
+      </geometry>
+    </collision>
   </link>
   <joint name="gear2_joint" type="revolute">
@@ -133,7 +200,8 @@
     <axis xyz="1 0 0"/>
     <mimic joint="gear1_joint" multiplier="-1.0" offset="0.0"/>
-    <limit lower="${-pi/2}" upper="${pi/2}" effort="100" velocity="1"/>
+    <limit lower="${-PI/2}" upper="${PI/2}" effort="${effort}" velocity="${velocity}"/>
   </joint>
   <link name="finger1_link">
+    <xacro:default_inertial mass="0.01"/>
     <visual>
       <origin xyz="0.03 0.24 -4.03" rpy="0 0 0"/>
@@ -143,4 +211,10 @@
       <material name="orange"/>
     </visual>
+    <collision>
+      <origin xyz="0 0 0" rpy="0 0 0"/>
+      <geometry>
+        <mesh filename="package://roboticarm_description/meshes/Gripper_1.001.stl" scale="0.01 0.01 0.01"/>
+      </geometry>
+    </collision>
   </link>
   <joint name="finger1_joint" type="fixed">
@@ -149,7 +223,8 @@
     <origin xyz="-0.055 -0.137 0.279" rpy="0 0 0"/>
     <axis xyz="0 1 0"/>
-    <limit lower="${-pi/2}" upper="${pi/2}" effort="100" velocity="1"/>
+    <limit lower="${-PI/2}" upper="${PI/2}" effort="${effort}" velocity="${velocity}"/>
   </joint>
   <link name="finger2_link">
+    <xacro:default_inertial mass="0.01"/>
     <visual>
       <origin xyz="0.03 -0.328 -4.01" rpy="0 0 0"/>
@@ -159,4 +234,10 @@
       <material name="orange"/>
     </visual>
+    <collision>
+      <origin xyz="0 0 0" rpy="0 0 0"/>
+      <geometry>
+        <mesh filename="package://roboticarm_description/meshes/Gripper_1.stl" scale="0.01 0.01 0.01"/>
+      </geometry>
+    </collision>
   </link>
   <joint name="finger2_joint" type="fixed">
@@ -165,5 +246,5 @@
     <origin xyz="-0.055 0.162 0.26" rpy="0 0 0"/>
     <axis xyz="0 1 0"/>
-    <limit lower="${-pi/2}" upper="${pi/2}" effort="100" velocity="1"/>
+    <limit lower="${-PI/2}" upper="${PI/2}" effort="${effort}" velocity="${velocity}"/>
   </joint>
 </robot>
